File: power-breakout.kicad_sch (KiCad schematic)
At the start: 13 parts, among them J1 Conn_02x08_Odd_Even, J2 Conn_02x05_Odd_Even, J3 Conn_01x03_Male, J4 Conn_02x04_Odd_Even, J5 Conn_02x04_Odd_Even

Commit message: adding BoM
Parts:
- J1: PartNum (none) -> A-2956; Vendor (none) -> Tayda
- J2: PartNum (none) -> A-2939; Vendor (none) -> Tayda
- J4, J5: PartNum (none) -> A-198; Vendor (none) -> Tayda
